Commit message: se agrega tf de footprint

File: urdf/bender.xacro (robot description, xacro)
@@ -25,4 +25,10 @@
   </collision>
 </link>
+<link name="base_footprint"/>
+<joint name="base_footprint_joint" type="fixed">
+  <parent link="base_footprint"/>
+  <child link="base_link"/>
+  <origin xyz="0 0 0.1" rpy="0 0 0"/>
+</joint>
 <link name="l2l_1">
   <inertial>
@@ -421,5 +427,5 @@
   </collision>
 </link>
-<link name="laser_1">
+<link name="laser">
   <inertial>
     <origin xyz="0.00021452729941068283 1.2832545766421587e-05 0.03715423693922987" rpy="0 0 0"/>

Commit message: (FG): added bender footprint tf for nav2

File: urdf/bender.xacro (robot description, xacro)
@@ -27,7 +27,7 @@
 <link name="base_footprint"/>
 <joint name="base_footprint_joint" type="fixed">
-  <parent link="base_footprint"/>
-  <child link="base_link"/>
-  <origin xyz="0 0 0.1" rpy="0 0 0"/>
+  <parent link="base_link"/>
+  <child link="base_footprint"/>
+  <origin xyz="0 0 0" rpy="0 0 0"/>
 </joint>
 <link name="l2l_1">
